Commit message: Port turtlebot3_lime to ROS 2 Jazzy / Ignition Gazebo (Harmonic)
## 動作確認済み機能
- Ignition Gazebo (Harmonic) でのロボット起動・シミュレーション
- MoveIt 2: アーム (joint1–6) の軌道計画・実行
- グリッパー (gripper_left/right_joint) の開閉制御
- Navigation2: SLAM マッピング・AMCL 自己位置推定・自律ナビゲーション
- MoveIt + Navigation2 統合起動 (moveit_navigation_use_sim_time.launch.py)

## 起動コマンド
# Gazebo シミュレーション
ros2 launch turtlebot3_lime_bringup gazebo.launch.py

# MoveIt のみ
ros2 launch turtlebot3_lime_moveit_config moveit_gazebo.launch.py

# Navigation2 のみ (map_yaml_file 指定)
ros2 launch turtlebot3_lime_navigation2 navigation2_use_sim_time.launch.py map_yaml_file:=<path>

# MoveIt + Navigation2 統合
ros2 launch turtlebot3_lime_bringup moveit_navigation_use_sim_time.launch.py map_yaml_file:=<path>

## 主な変更点 (Humble → Jazzy)
### Gazebo
- Classic Gazebo → Ignition Gazebo (Harmonic) へ移行
- gz_ros2_control/GazeboSimSystem プラグインに変更
- ros_gz_bridge による clock/odom/tf/scan/cmd_vel/camera ブリッジ設定追加
- SDF world ファイルを Ignition 形式に更新

### ros2_control / グリッパー
- gripper_left_joint: effort → position command interface
- gripper_right_joint: ros2_control mimic param でスレーブ制御
- URDF: gripper dynamics の friction 除去 (friction がDARTで関節をリセットしていた)
- コントローラー: position_controllers/GripperActionController に変更

### MoveIt 2
- OMPL プランニングパイプラインを Jazzy API に対応
- joint_limits.yaml の acceleration limits を robot_description_planning namespace に移動
- allowed_goal_duration_margin: 0.5 → 2.0 s (gripper stall_timeout 考慮)
- moveit_rviz.launch.py: RViz ログレベルを WARN に設定

### Navigation2 (Jazzy Nav2 1.3.x 対応)
- bt_navigator: plugin_lib_names リスト廃止 → navigators プラグイン構造に変更
- controller_server: progress_checker_plugin → progress_checker_plugins (複数形)
- behavior_server: プラグイン名 nav2_behaviors/Spin → nav2_behaviors::Spin
- planner_server: nav2_navfn_planner/NavfnPlanner → nav2_navfn_planner::NavfnPlanner
- collision_monitor: Jazzy 新規ライフサイクルノード、設定追加
- docking_server: Jazzy 新規ライフサイクルノード、設定追加
- launch: 廃止された default_bt_xml_filename 引数を削除、log_level 引数追加

## Future Work
- グリッパー把持シミュレーション (gz-sim-detachable-joint-system)
- Navigation2 統合テスト拡充

Co-Authored-By: Claude Sonnet 4.6 <noreply@anthropic.com>

File: turtlebot3_lime_description/gazebo/open_manipulator_sara.gazebo.xacro (robot description, xacro)
@@ -1,53 +1,25 @@
 <?xml version="1.0"?>
-<!--
-Copied and modified from turtlebot3 example:
-https://github.com/ROBOTIS-GIT/turtlebot3/blob/kinetic-devel/turtlebot3_description/urdf/turtlebot3_waffle_pi_for_open_manipulator.gazebo.xacro
--->
 <robot xmlns:xacro="http://ros.org/wiki/xacro">
   <xacro:macro name="open_manipulator_sara_gazebo" params="prefix">
-  <xacro:macro name="SimpleTransmission" params="trans joint actuator">
-    <transmission name="${trans}">
-      <type>transmission_interface/SimpleTransmission</type>
-      <joint name="${joint}">
-        <hardwareInterface>PositionJointInterface</hardwareInterface>
-      </joint>
-      <actuator name="${actuator}">
-        <mechanicalReduction>1</mechanicalReduction>
-        <hardwareInterface>PositionJointInterface</hardwareInterface>
-      </actuator>
-    </transmission>
-    <gazebo reference="${joint}">
-      <implicitSpringDamper>true</implicitSpringDamper>
-    </gazebo>
-  </xacro:macro>
-  <xacro:macro name="Link" params="reference">
-    <gazebo reference="${reference}">
-      <kp>1000000.0</kp>
-      <kd>100.0</kd>
-      <mu1>30.0</mu1>
-      <mu2>30.0</mu2>
-      <maxVel>1.0</maxVel>
-      <minDepth>0.001</minDepth>
-      <material>Gazebo/DarkGrey</material>
-    </gazebo>
-  </xacro:macro>
-  <xacro:Link reference="${prefix}link1"/>
-  <xacro:Link reference="${prefix}link2"/>
-  <xacro:Link reference="${prefix}link3"/>
-  <xacro:Link reference="${prefix}link4"/>
-  <xacro:Link reference="${prefix}link5"/>
-  <xacro:Link reference="${prefix}link6"/>
-  <xacro:Link reference="${prefix}link7"/>
-  <xacro:Link reference="${prefix}gripper_left_link"/>
-  <xacro:Link reference="${prefix}gripper_right_link"/>
-  <gazebo reference="${prefix}end_effector_link">
-    <material>Gazebo/Red</material>
-  </gazebo>
-  <xacro:SimpleTransmission trans="${prefix}trans1" joint="${prefix}joint1" actuator="${prefix}actuator1" />
-  <xacro:SimpleTransmission trans="${prefix}trans2" joint="${prefix}joint2" actuator="${prefix}actuator2" />
-  <xacro:SimpleTransmission trans="${prefix}trans3" joint="${prefix}joint3" actuator="${prefix}actuator3" />
-  <xacro:SimpleTransmission trans="${prefix}trans4" joint="${prefix}joint4" actuator="${prefix}actuator4" />
-  <xacro:SimpleTransmission trans="${prefix}trans5" joint="${prefix}gripper_left_joint" actuator="${prefix}actuator5" />
-  <xacro:SimpleTransmission trans="${prefix}trans6" joint="${prefix}gripper_right_joint" actuator="${prefix}actuator6" />
+    <!-- Link contact/friction properties (classic-compatible, used for ODE physics) -->
+    <xacro:macro name="Link" params="reference">
+      <gazebo reference="${reference}">
+        <kp>1000000.0</kp>
+        <kd>100.0</kd>
+        <mu1>30.0</mu1>
+        <mu2>30.0</mu2>
+        <maxVel>1.0</maxVel>
+        <minDepth>0.001</minDepth>
+      </gazebo>
+    </xacro:macro>
+    <xacro:Link reference="${prefix}link1"/>
+    <xacro:Link reference="${prefix}link2"/>
+    <xacro:Link reference="${prefix}link3"/>
+    <xacro:Link reference="${prefix}link4"/>
+    <xacro:Link reference="${prefix}link5"/>
+    <xacro:Link reference="${prefix}link6"/>
+    <xacro:Link reference="${prefix}link7"/>
+    <xacro:Link reference="${prefix}gripper_left_link"/>
+    <xacro:Link reference="${prefix}gripper_right_link"/>
   </xacro:macro>
 </robot>

File: turtlebot3_lime_description/gazebo/turtlebot3_bigwheel_orin.gazebo.xacro (robot description, xacro)
@@ -1,15 +1,8 @@
 <?xml version="1.0"?>
-<!--
-Copied and modified from turtlebot3 example:
-https://github.com/ROBOTIS-GIT/turtlebot3/blob/kinetic-devel/turtlebot3_description/urdf/turtlebot3_waffle_pi_for_open_manipulator.gazebo.xacro
--->
 <robot xmlns:xacro="http://ros.org/wiki/xacro">
   <xacro:macro name="turtlebot3_bigwheel_orin_gazebo" params="prefix">
     <xacro:property name="laser_visual" value="true"/>
-    <xacro:property name="camera_visual" value="true"/>
     <xacro:property name="imu_visual" value="true"/>
-    <gazebo reference="${prefix}base_link">
-      <material>Gazebo/DarkGrey</material>
-    </gazebo>
+    <!-- Wheel contact/friction properties -->
     <gazebo reference="${prefix}wheel_left_link">
       <mu1>1.0</mu1>
@@ -20,5 +13,4 @@
       <maxVel>0.1</maxVel>
       <fdir1>1 0 0</fdir1>
-      <material>Gazebo/Green</material>
     </gazebo>
     <gazebo reference="${prefix}wheel_right_link">
@@ -30,5 +22,4 @@
       <maxVel>0.1</maxVel>
       <fdir1>1 0 0</fdir1>
-      <material>Gazebo/Green</material>
     </gazebo>
     <gazebo reference="${prefix}caster_back_right_link">
@@ -39,5 +30,4 @@
       <minDepth>0.001</minDepth>
       <maxVel>1.0</maxVel>
-      <material>Gazebo/FlatBlack</material>
     </gazebo>
     <gazebo reference="${prefix}caster_back_left_link">
@@ -48,46 +38,63 @@
       <minDepth>0.001</minDepth>
       <maxVel>1.0</maxVel>
-      <material>Gazebo/FlatBlack</material>
     </gazebo>
+    <!-- IMU sensor (Ignition Gazebo) -->
     <gazebo reference="${prefix}imu_link">
-      <material>Gazebo/Grey</material>
-      <sensor type="imu" name="imu">
+      <sensor name="tb3_imu" type="imu">
         <always_on>true</always_on>
-        <update_rate>100.0</update_rate>
-        <visualize>${imu_visual}</visualize>
+        <update_rate>200</update_rate>
+        <topic>imu</topic>
+        <gz_frame_id>${prefix}imu_link</gz_frame_id>
+        <imu>
+          <angular_velocity>
+            <x><noise type="gaussian"><mean>0.0</mean><stddev>2e-4</stddev></noise></x>
+            <y><noise type="gaussian"><mean>0.0</mean><stddev>2e-4</stddev></noise></y>
+            <z><noise type="gaussian"><mean>0.0</mean><stddev>2e-4</stddev></noise></z>
+          </angular_velocity>
+          <linear_acceleration>
+            <x><noise type="gaussian"><mean>0.0</mean><stddev>1.7e-2</stddev></noise></x>
+            <y><noise type="gaussian"><mean>0.0</mean><stddev>1.7e-2</stddev></noise></y>
+            <z><noise type="gaussian"><mean>0.0</mean><stddev>1.7e-2</stddev></noise></z>
+          </linear_acceleration>
+        </imu>
       </sensor>
     </gazebo>
+    <!-- Differential drive plugin (Ignition Gazebo) -->
     <gazebo>
-      <plugin name='diff_drive' filename='libgazebo_ros_diff_drive.so'>
-        <ros>
-          <namespace></namespace>
-          <remapping>cmd_vel:=cmd_vel</remapping>
-          <remapping>odom:=odom</remapping>
-        </ros>
-        <left_joint>wheel_left_joint</left_joint>
-        <right_joint>wheel_right_joint</right_joint>
+      <plugin filename="gz-sim-diff-drive-system" name="gz::sim::systems::DiffDrive">
+        <left_joint>${prefix}wheel_left_joint</left_joint>
+        <right_joint>${prefix}wheel_right_joint</right_joint>
         <wheel_separation>0.29425</wheel_separation>
-        <wheel_diameter>0.12</wheel_diameter>
-        <max_wheel_torque>20</max_wheel_torque>
-        <max_wheel_acceleration>1.0</max_wheel_acceleration>
-        <publish_odom>true</publish_odom>
-        <publish_odom_tf>true</publish_odom_tf>
-        <publish_wheel_tf>false</publish_wheel_tf>
-        <odometry_frame>odom</odometry_frame>
-        <robot_base_frame>base_footprint</robot_base_frame>
+        <wheel_radius>0.06</wheel_radius>
+        <max_linear_acceleration>1.0</max_linear_acceleration>
+        <topic>cmd_vel</topic>
+        <odom_topic>odom</odom_topic>
+        <frame_id>odom</frame_id>
+        <child_frame_id>${prefix}base_footprint</child_frame_id>
+        <odom_publisher_frequency>30</odom_publisher_frequency>
+        <tf_topic>/tf</tf_topic>
       </plugin>
     </gazebo>
+    <!-- Wheel joint states (Ignition Gazebo) -->
+    <gazebo>
+      <plugin filename="gz-sim-joint-state-publisher-system" name="gz::sim::systems::JointStatePublisher">
+        <topic>joint_states</topic>
+        <joint_name>${prefix}wheel_left_joint</joint_name>
+        <joint_name>${prefix}wheel_right_joint</joint_name>
+      </plugin>
+    </gazebo>
+    <!-- LiDAR sensor (Ignition Gazebo gpu_lidar) -->
     <gazebo reference="${prefix}base_scan">
-      <material>Gazebo/FlatBlack</material>
-      <sensor type="ray" name="lds_lfcd_sensor">
-        <pose>0 0 0 0 0 0</pose>
+      <sensor name="hls_lfcd_lds" type="gpu_lidar">
         <always_on>true</always_on>
-        <update_rate>5.0</update_rate>
         <visualize>${laser_visual}</visualize>
-        <ray>
+        <update_rate>5</update_rate>
+        <topic>scan</topic>
+        <gz_frame_id>${prefix}base_scan</gz_frame_id>
+        <lidar>
           <scan>
             <horizontal>
               <samples>360</samples>
-              <resolution>1</resolution>
+              <resolution>1.0</resolution>
               <min_angle>0.0</min_angle>
               <max_angle>6.28319</max_angle>
@@ -104,35 +111,20 @@
             <stddev>0.01</stddev>
           </noise>
-        </ray>
-        <plugin name="gazebo_ros_lds_lfcd_controller" filename="libgazebo_ros_ray_sensor.so">
-          <ros>
-            <namespace></namespace>
-            <remapping>~/out:=scan</remapping>
-          </ros>
-          <output_type>sensor_msgs/LaserScan</output_type>
-        </plugin>
+        </lidar>
       </sensor>
     </gazebo>
+    <!-- RGBD camera sensor (Ignition Gazebo, replaces librealsense_gazebo_plugin) -->
     <gazebo reference="camera_link">
-      <self_collide>0</self_collide>
-      <enable_wind>0</enable_wind>
-      <kinematic>0</kinematic>
-      <gravity>1</gravity>
-      <!--<mu>1</mu>-->
-      <mu2>1</mu2>
-      <fdir1>0 0 0</fdir1>
-      <!--<slip1>0</slip1>
-      <slip2>0</slip2>-->
-      <kp>1e+13</kp>
-      <kd>1</kd>
-      <!--<max_vel>0.01</max_vel>
-      <min_depth>0</min_depth>-->
-      <sensor name="cameracolor" type="camera">
-        <camera name="camera">
+      <sensor name="depth_camera" type="rgbd_camera">
+        <always_on>true</always_on>
+        <update_rate>30</update_rate>
+        <topic>camera</topic>
+        <gz_frame_id>camera_link</gz_frame_id>
+        <camera>
           <horizontal_fov>1.2112585008840648</horizontal_fov>
           <image>
             <width>640</width>
             <height>480</height>
-            <format>RGB_INT8</format>
+            <format>R8G8B8</format>
           </image>
           <clip>
@@ -146,99 +138,5 @@
           </noise>
         </camera>
-        <always_on>1</always_on>
-        <update_rate>30</update_rate>
-        <visualize>1</visualize>
       </sensor>
-      <sensor name="cameraired1" type="camera">
-        <camera name="camera">
-          <horizontal_fov>1.4870205226991688</horizontal_fov>
-          <image>
-            <width>640</width>
-            <height>480</height>
-            <format>L_INT8</format>
-          </image>
-          <clip>
-            <near>0.1</near>
-            <far>100</far>
-          </clip>
-          <noise>
-            <type>gaussian</type>
-            <mean>0.0</mean>
-            <stddev>0.05</stddev>
-          </noise>
-        </camera>
-        <always_on>1</always_on>
-        <update_rate>90</update_rate>
-        <visualize>0</visualize>
-      </sensor>
-      <sensor name="cameraired2" type="camera">
-        <camera name="camera">
-          <horizontal_fov>1.4870205226991688</horizontal_fov>
-          <image>
-            <width>640</width>
-            <height>480</height>
-            <format>L_INT8</format>
-          </image>
-          <clip>
-            <near>0.1</near>
-            <far>100</far>
-          </clip>
-          <noise>
-            <type>gaussian</type>
-            <mean>0.0</mean>
-            <stddev>0.05</stddev>
-          </noise>
-        </camera>
-        <always_on>1</always_on>
-        <update_rate>90</update_rate>
-        <visualize>0</visualize>
-      </sensor>
-      <sensor name="cameradepth" type="depth">
-        <camera name="camera">
-          <horizontal_fov>1.4870205226991688</horizontal_fov>
-          <image>
-            <width>640</width>
-            <height>480</height>
-          </image>
-          <clip>
-            <near>0.1</near>
-            <far>100</far>
-          </clip>
-          <noise>
-            <type>gaussian</type>
-            <mean>0.0</mean>
-            <stddev>0.100</stddev>
-          </noise>
-        </camera>
-        <always_on>1</always_on>
-        <update_rate>90</update_rate>
-        <visualize>0</visualize>
-      </sensor>
-    </gazebo>
-    <gazebo>
-      <plugin filename="librealsense_gazebo_plugin.so" name="camera">
-        <prefix>camera</prefix>
-        <depthUpdateRate>30.0</depthUpdateRate>
-        <colorUpdateRate>30.0</colorUpdateRate>
-        <infraredUpdateRate>30.0</infraredUpdateRate>
-        <depthTopicName>camera/camera/depth/image_rect_raw</depthTopicName>
-        <depthCameraInfoTopicName>camera/camera/depth/camera_info</depthCameraInfoTopicName>
-        <colorTopicName>camera/camera/color/image_raw</colorTopicName>
-        <colorCameraInfoTopicName>camera/camera/color/camera_info</colorCameraInfoTopicName>
-        <infrared1TopicName>camera/camera/infra1/image_rect_raw</infrared1TopicName>
-        <infrared1CameraInfoTopicName>camera/camera/infra1/camera_info</infrared1CameraInfoTopicName>
-        <infrared2TopicName>camera/camera/infra2/image_rect_raw</infrared2TopicName>
-        <infrared2CameraInfoTopicName>camera/camera/infra2/camera_info</infrared2CameraInfoTopicName>
-        <colorOpticalframeName>camera_color_optical_frame</colorOpticalframeName>
-        <depthOpticalframeName>camera_depth_optical_frame</depthOpticalframeName>
-        <infrared1OpticalframeName>camera_infra1_optical_frame</infrared1OpticalframeName>
-        <infrared2OpticalframeName>camera_infra2_optical_frame</infrared2OpticalframeName>
-        <rangeMinDepth>0.2</rangeMinDepth>
-        <rangeMaxDepth>10.0</rangeMaxDepth>
-        <pointCloud>True</pointCloud>
-        <pointCloudTopicName>camera/camera/depth/color/points</pointCloudTopicName>
-        <pointCloudCutoff>0.25</pointCloudCutoff>
-        <pointCloudCutoffMax>9.0</pointCloudCutoffMax>
-      </plugin>
     </gazebo>
   </xacro:macro>
