Commit message: Port turtlebot3_lime to ROS 2 Jazzy / Ignition Gazebo (Harmonic)
## 動作確認済み機能
- Ignition Gazebo (Harmonic) でのロボット起動・シミュレーション
- MoveIt 2: アーム (joint1–6) の軌道計画・実行
- グリッパー (gripper_left/right_joint) の開閉制御
- Navigation2: SLAM マッピング・AMCL 自己位置推定・自律ナビゲーション
- MoveIt + Navigation2 統合起動 (moveit_navigation_use_sim_time.launch.py)

## 起動コマンド
# Gazebo シミュレーション
ros2 launch turtlebot3_lime_bringup gazebo.launch.py

# MoveIt のみ
ros2 launch turtlebot3_lime_moveit_config moveit_gazebo.launch.py

# Navigation2 のみ (map_yaml_file 指定)
ros2 launch turtlebot3_lime_navigation2 navigation2_use_sim_time.launch.py map_yaml_file:=<path>

# MoveIt + Navigation2 統合
ros2 launch turtlebot3_lime_bringup moveit_navigation_use_sim_time.launch.py map_yaml_file:=<path>

## 主な変更点 (Humble → Jazzy)
### Gazebo
- Classic Gazebo → Ignition Gazebo (Harmonic) へ移行
- gz_ros2_control/GazeboSimSystem プラグインに変更
- ros_gz_bridge による clock/odom/tf/scan/cmd_vel/camera ブリッジ設定追加
- SDF world ファイルを Ignition 形式に更新

### ros2_control / グリッパー
- gripper_left_joint: effort → position command interface
- gripper_right_joint: ros2_control mimic param でスレーブ制御
- URDF: gripper dynamics の friction 除去 (friction がDARTで関節をリセットしていた)
- コントローラー: position_controllers/GripperActionController に変更

### MoveIt 2
- OMPL プランニングパイプラインを Jazzy API に対応
- joint_limits.yaml の acceleration limits を robot_description_planning namespace に移動
- allowed_goal_duration_margin: 0.5 → 2.0 s (gripper stall_timeout 考慮)
- moveit_rviz.launch.py: RViz ログレベルを WARN に設定

### Navigation2 (Jazzy Nav2 1.3.x 対応)
- bt_navigator: plugin_lib_names リスト廃止 → navigators プラグイン構造に変更
- controller_server: progress_checker_plugin → progress_checker_plugins (複数形)
- behavior_server: プラグイン名 nav2_behaviors/Spin → nav2_behaviors::Spin
- planner_server: nav2_navfn_planner/NavfnPlanner → nav2_navfn_planner::NavfnPlanner
- collision_monitor: Jazzy 新規ライフサイクルノード、設定追加
- docking_server: Jazzy 新規ライフサイクルノード、設定追加
- launch: 廃止された default_bt_xml_filename 引数を削除、log_level 引数追加

## Future Work
- グリッパー把持シミュレーション (gz-sim-detachable-joint-system)
- Navigation2 統合テスト拡充

Co-Authored-By: Claude Sonnet 4.6 <noreply@anthropic.com>

File: turtlebot3_lime_description/ros2_control/turtlebot3_lime_system.ros2_control.xacro (robot description, xacro)
@@ -1,8 +1,3 @@
 <?xml version="1.0"?>
-<!--
-Copied and modified from ros2 control demos example:
-https://github.com/ros-controls/ros2_control_demos/blob/foxy/ros2_control_demo_description/diffbot_description/ros2_control/diffbot_system.ros2_control.xacro
-https://github.com/ros-controls/ros2_control_demos/blob/foxy/ros2_control_demo_description/rrbot_description/ros2_control/rrbot_system_position_only.ros2_control.xacro
--->
 <robot xmlns:xacro="http://www.ros.org/wiki/xacro">
   <xacro:macro name="turtlebot3_lime_system" params="name prefix use_sim:=^|false use_fake_hardware:=^|false fake_sensor_commands:=^|false">
@@ -10,5 +5,5 @@
       <xacro:if value="$(arg use_sim)">
         <hardware>
-          <plugin>gazebo_ros2_control/GazeboSystem</plugin>
+          <plugin>gz_ros2_control/GazeboSimSystem</plugin>
         </hardware>
       </xacro:if>
@@ -16,5 +11,5 @@
         <hardware>
           <xacro:if value="${use_fake_hardware}">
-            <plugin>fake_components/GenericSystem</plugin>
+            <plugin>mock_components/GenericSystem</plugin>
             <param name="fake_sensor_commands">${fake_sensor_commands}</param>
             <param name="state_following_offset">0.0</param>
@@ -32,74 +27,79 @@
         </hardware>
       </xacro:unless>
-      <joint name="${prefix}wheel_left_joint">
-        <command_interface name="velocity">
-          <param name="min">-24.5</param>
-          <param name="max">24.5</param>
-        </command_interface>
-        <state_interface name="position">
-          <param name="initial_value">0.0</param>
-        </state_interface>
-        <state_interface name="velocity">
-          <param name="initial_value">0.0</param>
-        </state_interface>
-      </joint>
-      <joint name="${prefix}wheel_right_joint">
-        <command_interface name="velocity">
-          <param name="min">-24.5</param>
-          <param name="max">24.5</param>
-        </command_interface>
-        <state_interface name="position">
-          <param name="initial_value">0.0</param>
-        </state_interface>
-        <state_interface name="velocity">
-          <param name="initial_value">0.0</param>
-        </state_interface>
-      </joint>
-      <sensor name="imu">
-        <state_interface name="orientation.x">
-          <param name="initial_value">0.0</param>
-        </state_interface>
-        <state_interface name="orientation.y">
-          <param name="initial_value">0.0</param>
-        </state_interface>
-        <state_interface name="orientation.z">
-          <param name="initial_value">0.0</param>
-        </state_interface>
-        <state_interface name="orientation.w">
-          <param name="initial_value">0.0</param>
-        </state_interface>
-        <state_interface name="angular_velocity.x">
-          <param name="initial_value">0.0</param>
-        </state_interface>
-        <state_interface name="angular_velocity.y">
-          <param name="initial_value">0.0</param>
-        </state_interface>
-        <state_interface name="angular_velocity.z">
-          <param name="initial_value">0.0</param>
-        </state_interface>
-        <state_interface name="linear_acceleration.x">
-          <param name="initial_value">0.0</param>
-        </state_interface>
-        <state_interface name="linear_acceleration.y">
-          <param name="initial_value">0.0</param>
-        </state_interface>
-        <state_interface name="linear_acceleration.z">
-          <param name="initial_value">0.0</param>
-        </state_interface>
-      </sensor>
-      <sensor name="battery">
-        <state_interface name="voltage">
-          <param name="initial_value">0.0</param>
-        </state_interface>
-        <state_interface name="percentage">
-          <param name="initial_value">0.0</param>
-        </state_interface>
-        <state_interface name="design_capacity">
-          <param name="initial_value">0.0</param>
-        </state_interface>
-        <state_interface name="present">
-          <param name="initial_value">0.0</param>
-        </state_interface>
-      </sensor>
+      <!-- Wheel joints and hardware sensors: excluded when use_sim=true.
+           Wheels are driven by gz-sim-diff-drive-system; IMU/battery are hardware-only. -->
+      <xacro:unless value="$(arg use_sim)">
+        <joint name="${prefix}wheel_left_joint">
+          <command_interface name="velocity">
+            <param name="min">-24.5</param>
+            <param name="max">24.5</param>
+          </command_interface>
+          <state_interface name="position">
+            <param name="initial_value">0.0</param>
+          </state_interface>
+          <state_interface name="velocity">
+            <param name="initial_value">0.0</param>
+          </state_interface>
+        </joint>
+        <joint name="${prefix}wheel_right_joint">
+          <command_interface name="velocity">
+            <param name="min">-24.5</param>
+            <param name="max">24.5</param>
+          </command_interface>
+          <state_interface name="position">
+            <param name="initial_value">0.0</param>
+          </state_interface>
+          <state_interface name="velocity">
+            <param name="initial_value">0.0</param>
+          </state_interface>
+        </joint>
+        <sensor name="tb3_imu">
+          <state_interface name="orientation.x">
+            <param name="initial_value">0.0</param>
+          </state_interface>
+          <state_interface name="orientation.y">
+            <param name="initial_value">0.0</param>
+          </state_interface>
+          <state_interface name="orientation.z">
+            <param name="initial_value">0.0</param>
+          </state_interface>
+          <state_interface name="orientation.w">
+            <param name="initial_value">0.0</param>
+          </state_interface>
+          <state_interface name="angular_velocity.x">
+            <param name="initial_value">0.0</param>
+          </state_interface>
+          <state_interface name="angular_velocity.y">
+            <param name="initial_value">0.0</param>
+          </state_interface>
+          <state_interface name="angular_velocity.z">
+            <param name="initial_value">0.0</param>
+          </state_interface>
+          <state_interface name="linear_acceleration.x">
+            <param name="initial_value">0.0</param>
+          </state_interface>
+          <state_interface name="linear_acceleration.y">
+            <param name="initial_value">0.0</param>
+          </state_interface>
+          <state_interface name="linear_acceleration.z">
+            <param name="initial_value">0.0</param>
+          </state_interface>
+        </sensor>
+        <sensor name="battery">
+          <state_interface name="voltage">
+            <param name="initial_value">0.0</param>
+          </state_interface>
+          <state_interface name="percentage">
+            <param name="initial_value">0.0</param>
+          </state_interface>
+          <state_interface name="design_capacity">
+            <param name="initial_value">0.0</param>
+          </state_interface>
+          <state_interface name="present">
+            <param name="initial_value">0.0</param>
+          </state_interface>
+        </sensor>
+      </xacro:unless>
+      <!-- Arm joints: always present (gz_ros2_control/GazeboSimSystem manages these in sim) -->
       <joint name="${prefix}joint1">
         <command_interface name="position">
@@ -116,5 +116,29 @@
       <joint name="${prefix}joint2">
         <command_interface name="position">
-          <param name="min">${-pi*0.57}</param>
+          <param name="min">${-pi*0.541}</param>
+          <param name="max">${pi*0.562}</param>
+        </command_interface>
+        <state_interface name="position">
+          <param name="initial_value">0.0</param>
+        </state_interface>
+        <state_interface name="velocity">
+          <param name="initial_value">0.0</param>
+        </state_interface>
+      </joint>
+      <joint name="${prefix}joint3">
+        <command_interface name="position">
+          <param name="min">${-pi*0.560}</param>
+          <param name="max">${pi*0.591}</param>
+        </command_interface>
+        <state_interface name="position">
+          <param name="initial_value">0.0</param>
+        </state_interface>
+        <state_interface name="velocity">
+          <param name="initial_value">0.0</param>
+        </state_interface>
+      </joint>
+      <joint name="${prefix}joint4">
+        <command_interface name="position">
+          <param name="min">${-pi*0.5}</param>
           <param name="max">${pi*0.5}</param>
         </command_interface>
@@ -126,32 +150,8 @@
         </state_interface>
       </joint>
-      <joint name="${prefix}joint3">
-        <command_interface name="position">
-          <param name="min">${-pi*0.3}</param>
-          <param name="max">${pi*0.44}</param>
-        </command_interface>
-        <state_interface name="position">
-          <param name="initial_value">0.0</param>
-        </state_interface>
-        <state_interface name="velocity">
-          <param name="initial_value">0.0</param>
-        </state_interface>
-      </joint>
-      <joint name="${prefix}joint4">
-        <command_interface name="position">
-          <param name="min">${-pi*0.57}</param>
-          <param name="max">${pi*0.65}</param>
-        </command_interface>
-        <state_interface name="position">
-          <param name="initial_value">0.0</param>
-        </state_interface>
-        <state_interface name="velocity">
-          <param name="initial_value">0.0</param>
-        </state_interface>
-      </joint>
       <joint name="${prefix}joint5">
         <command_interface name="position">
-          <param name="min">${-pi*0.57}</param>
-          <param name="max">${pi*0.65}</param>
+          <param name="min">${-pi*0.531}</param>
+          <param name="max">${pi*0.567}</param>
         </command_interface>
         <state_interface name="position">
@@ -164,6 +164,6 @@
       <joint name="${prefix}joint6">
         <command_interface name="position">
-          <param name="min">${-pi*0.57}</param>
-          <param name="max">${pi*0.65}</param>
+          <param name="min">${-pi*0.9}</param>
+          <param name="max">${pi*0.9}</param>
         </command_interface>
         <state_interface name="position">
@@ -189,8 +189,4 @@
         <param name="mimic">gripper_left_joint</param>
         <param name="multiplier">1</param>
-        <command_interface name="position">
-          <param name="min">-0.010</param>
-          <param name="max">0.019</param>
-        </command_interface>
         <state_interface name="position">
           <param name="initial_value">0.0</param>

File: turtlebot3_lime_description/urdf/open_manipulator_sara.urdf.xacro (robot description, xacro)
@@ -61,6 +61,6 @@
       <origin xyz="0.0 0.0 0.0595" rpy="0 0 0"/>
       <axis xyz="0 1 0"/>
-      <limit velocity="4.8" effort="1" lower="${-pi*0.541}" upper="${pi*0.562}" />
-      <dynamics damping="0.7" friction="1.0"/>
+      <limit velocity="4.8" effort="100" lower="${-pi*0.541}" upper="${pi*0.562}" />
+      <dynamics damping="0.1" friction="1.0"/>
     </joint>
     <link name="${prefix}link3">
@@ -163,9 +163,4 @@
       </collision>
       <inertial>
-        <origin xyz="0 0 0" />
-        <mass value="0.033" />
-        <inertia ixx="0.1" ixy="0.0" ixz="0.0" iyy="0.1" iyz="0.0" izz="0.1" />
-      </inertial>
-      <inertial>
         <origin xyz="4.4206755e-02 3.6839985e-07 8.9142216e-03" />
         <mass value="1.4327573e-01" />
@@ -226,6 +221,6 @@
       <origin xyz="0.0 0.021 0.0707" rpy="0 0 0"/>
       <axis xyz="0 1 0"/>
-      <limit velocity="4.8" effort="1" lower="-0.010" upper="0.019" />
-      <dynamics damping="0.7" friction="1.0"/>
+      <limit velocity="4.8" effort="1000" lower="-0.010" upper="0.019" />
+      <dynamics damping="0.1"/>
     </joint>
     <!-- Move it 2 not find mimic-->
@@ -241,7 +236,7 @@
       <origin xyz="0.0 -0.021 0.0707" rpy="0 0 0"/>
       <axis xyz="0 -1 0"/>
-      <limit velocity="4.8" effort="1" lower="-0.010" upper="0.019" />
+      <limit velocity="4.8" effort="1000" lower="-0.010" upper="0.019" />
       <mimic joint="${prefix}gripper_left_joint" multiplier="1"/>
-      <dynamics damping="0.7" friction="1.0"/>
+      <dynamics damping="0.1"/>
     </joint>
     <link name="${prefix}gripper_right_link">

File: turtlebot3_lime_description/urdf/turtlebot3_lime.urdf.xacro (robot description, xacro)
@@ -5,4 +5,5 @@
   <xacro:arg name="prefix" default="" />
   <xacro:arg name="use_sim" default="false" />
+  <xacro:arg name="gz_cm_yaml_path" default="$(find turtlebot3_lime_bringup)/config/gazebo_controller_manager.yaml" />
   <xacro:arg name="use_fake_hardware" default="false" />
   <xacro:arg name="fake_sensor_commands" default="false" />
@@ -31,6 +32,6 @@
   <xacro:turtlebot3_lime_system name="TurtleBot3LimeSystem" prefix="$(arg prefix)" use_sim="$(arg use_sim)" use_fake_hardware="$(arg use_fake_hardware)" fake_sensor_commands="$(arg fake_sensor_commands)"/>
   <gazebo>
-    <plugin name="gazebo_ros2_control" filename="libgazebo_ros2_control.so">
-      <parameters>$(find turtlebot3_lime_bringup)/config/gazebo_controller_manager.yaml</parameters>
+    <plugin filename="gz_ros2_control-system" name="gz_ros2_control::GazeboSimROS2ControlPlugin">
+      <parameters>$(arg gz_cm_yaml_path)</parameters>
     </plugin>
   </gazebo>
