Commit message: confirm gazebo.launch.py

File: turtlebot3_lime_description/gazebo/turtlebot3_bigwheel_orin.gazebo.xacro (robot description, xacro)
@@ -6,6 +6,6 @@
     <!-- Wheel contact/friction properties -->
     <gazebo reference="${prefix}wheel_left_link">
-      <mu1>1.0</mu1>
-      <mu2>1.0</mu2>
+      <mu1>1000.0</mu1>
+      <mu2>1000.0</mu2>
       <kp>500000.0</kp>
       <kd>10.0</kd>
@@ -15,6 +15,6 @@
     </gazebo>
     <gazebo reference="${prefix}wheel_right_link">
-      <mu1>1.0</mu1>
-      <mu2>1.0</mu2>
+      <mu1>1000.0</mu1>
+      <mu2>1000.0</mu2>
       <kp>500000.0</kp>
       <kd>10.0</kd>

File: turtlebot3_lime_description/urdf/open_manipulator_sara.urdf.xacro (robot description, xacro)
@@ -33,6 +33,6 @@
       <origin xyz="0.012 0.0 0.017" rpy="0 0 0"/>
       <axis xyz="0 0 1"/>
-      <limit velocity="4.8" effort="1" lower="${-pi*0.9}" upper="${pi*0.9}" />
-      <dynamics damping="0.7" friction="1.0"/>
+      <limit velocity="4.8" effort="100" lower="${-pi*0.9}" upper="${pi*0.9}" />
+      <dynamics damping="0.1" friction="1.0"/>
     </joint>
     <link name="${prefix}link2">
@@ -89,6 +89,6 @@
       <origin xyz="0.0 0 0.124" rpy="0 0 0"/>
       <axis xyz="0 1 0"/>
-      <limit velocity="4.8" effort="1" lower="${-pi*0.560}" upper="${pi*0.591}" />
-      <dynamics damping="0.7" friction="1.0"/>
+      <limit velocity="4.8" effort="100" lower="${-pi*0.560}" upper="${pi*0.591}" />
+      <dynamics damping="0.1" friction="1.0"/>
     </joint>
     <link name="${prefix}link4">
@@ -117,6 +117,6 @@
       <origin xyz="0.0 0.0 0.045" rpy="0 0 0"/>
       <axis xyz="0 0 1"/>
-      <limit velocity="4.8" effort="1" lower="${-pi*0.5}" upper="${pi*0.5}" />
-      <dynamics damping="0.7" friction="1.0"/>
+      <limit velocity="4.8" effort="100" lower="${-pi*0.5}" upper="${pi*0.5}" />
+      <dynamics damping="0.1" friction="1.0"/>
     </joint>
     <link name="${prefix}link5">
@@ -145,6 +145,6 @@
       <origin xyz="0.0 0.0 0.0595" rpy="0 0 0"/>
       <axis xyz="0 1 0"/>
-      <limit velocity="4.8" effort="1" lower="${-pi*0.531}" upper="${pi*0.567}" />
-      <dynamics damping="0.7" friction="1.0"/>
+      <limit velocity="4.8" effort="100" lower="${-pi*0.531}" upper="${pi*0.567}" />
+      <dynamics damping="0.1" friction="1.0"/>
     </joint>
     <link name="${prefix}link6">
@@ -173,6 +173,6 @@
       <origin xyz="0.0 0.0 0.0475" rpy="0 0 0"/>
       <axis xyz="0 0 1"/>
-      <limit velocity="4.8" effort="1" lower="${-pi*0.9}" upper="${pi*0.9}" />
-      <dynamics damping="0.7" friction="1.0"/>
+      <limit velocity="4.8" effort="100" lower="${-pi*0.9}" upper="${pi*0.9}" />
+      <dynamics damping="0.1" friction="1.0"/>
     </joint>
     <link name="${prefix}link7">
