Commit message: Tested and working(only arm)

File: turtlebot3_lime_description/urdf/open_manipulator_sara.urdf.xacro (robot description, xacro)
@@ -6,6 +6,9 @@
 -->
 <robot xmlns:xacro="http://www.ros.org/wiki/xacro">
+  <material name="grey">
+    <color rgba="0.5 0.5 0.5 1.0"/>
+  </material>
   <xacro:macro name="open_manipulator_sara" params="prefix">
-    <xacro:property name="meshes_file_direction" value="package://turtlebot3_lime_description/meshes/open_manipulator_sara"/>
+    <xacro:property name="meshes_file_direction" value="file://$(find turtlebot3_lime_description)/meshes/open_manipulator_sara"/>
     <link name="${prefix}link1">
       <visual>
@@ -61,6 +64,6 @@
       <origin xyz="0.0 0.0 0.0595" rpy="0 0 0"/>
       <axis xyz="0 1 0"/>
-      <limit velocity="4.8" effort="1" lower="${-pi*0.541}" upper="${pi*0.562}" />
-      <dynamics damping="0.7" friction="1.0"/>
+      <limit velocity="4.8" effort="100" lower="${-pi*0.541}" upper="${pi*0.562}" />
+      <dynamics damping="0.1" friction="1.0"/>
     </joint>
     <link name="${prefix}link3">
@@ -163,9 +166,4 @@
       </collision>
       <inertial>
-        <origin xyz="0 0 0" />
-        <mass value="0.033" />
-        <inertia ixx="0.1" ixy="0.0" ixz="0.0" iyy="0.1" iyz="0.0" izz="0.1" />
-      </inertial>
-      <inertial>
         <origin xyz="4.4206755e-02 3.6839985e-07 8.9142216e-03" />
         <mass value="1.4327573e-01" />
@@ -227,5 +225,5 @@
       <axis xyz="0 1 0"/>
       <limit velocity="4.8" effort="1" lower="-0.010" upper="0.019" />
-      <dynamics damping="0.7" friction="1.0"/>
+      <dynamics damping="0.1" friction="1.0"/>
     </joint>
     <!-- Move it 2 not find mimic-->
@@ -242,6 +240,5 @@
       <axis xyz="0 -1 0"/>
       <limit velocity="4.8" effort="1" lower="-0.010" upper="0.019" />
-      <mimic joint="${prefix}gripper_left_joint" multiplier="1"/>
-      <dynamics damping="0.7" friction="1.0"/>
+      <dynamics damping="0.1" friction="1.0"/>
     </joint>
     <link name="${prefix}gripper_right_link">

File: turtlebot3_lime_description/urdf/standalone_sara.urdf.xacro (robot description, xacro)
@@ -2,4 +2,6 @@
 <robot name="open_manipulator_sara" xmlns:xacro="http://ros.org/wiki/xacro">
   <xacro:include filename="$(find turtlebot3_lime_description)/urdf/open_manipulator_sara.urdf.xacro" />
+  <xacro:include filename="$(find turtlebot3_lime_description)/gazebo/open_manipulator_sara.gazebo.xacro" />
+  <xacro:include filename="$(find turtlebot3_lime_description)/ros2_control/open_manipulator_sara.ros2_control.xacro" />
   <xacro:arg name="prefix" default="" />
   <xacro:arg name="use_sim" default="true" />
